File: PlacaEletronica/Robo_opcao.brd (EAGLE design)
At the start: 139.7 x 148 mm, 101 parts, among them IC1 7805DT, IC2 7805DT, J1 F-1X06-SIP-100-40, J2 S2B-PH-K-S(LF)(SN), J3 ZX62-B-5PA, Q1 SMD-TRANSISTORS-NPN-25V-500MW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, Q2 SMD-TRANSISTORS-NPN-25V-500MW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, Q4 SFH_3716, U1 ESP32-WROOM-32D, U2 AMS1117-3.3, U3 INTERFACE-CP2102-GMR(QFN28)QF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

Commit message: Tudo funcionando perfeitamente antes de implementar upload OTA
Parts:
- moved R53 103.3 mm to (127.3, 89.7), turned to 0 degrees
- moved Q2 100.4 mm to (127.8, 93.8)
- moved R51 95.3 mm to (123.6, 88.4), turned to 0 degrees
- moved R52 93.9 mm to (123.6, 89.7), turned to 0 degrees
- moved Q1 90.6 mm to (123.9, 93.8), turned to 0 degrees
- moved U3 7.01 mm to (125.1, 107.4)
- moved J3 3.81 mm to (137.7, 104.5)
Routing:
- net SS: track 255.6 -> 157.5 mm, vias 1 -> 8
- net EN: track 96.8 -> 182.1 mm, vias 2 -> 4
- net DTR: track 129.6 -> 54.9 mm, vias 4 -> 0
- net 5_S: track 89.6 -> 162.2 mm, vias 3 -> 2
- net RX0: track 255.0 -> 324.1 mm, vias 7 -> 5
- net 7_S: track 233.3 -> 164.8 mm, vias 3 -> 4
- net MISO: track 192.7 -> 138.1 mm, vias 4 -> 8
- net B-: track 177.7 -> 230.2 mm, vias 6 -> 1
- net PORT_13~5V: track 149.4 -> 196.0 mm, vias 3 -> 6
- net 8_S: track 177.1 -> 133.5 mm, vias 6 -> 4
- net VP_SENSOR: track 177.5 -> 213.9 mm, vias 1 -> 3
- net MOSI: track 134.4 -> 168.6 mm, vias 2 -> 6
- net N$3: track 0.00 -> 34.1 mm, vias 0 -> 4
- net IO0: track 130.5 -> 101.1 mm, vias 2 -> 0
- net GND_PWM~5V: track 415.1 -> 387.7 mm, vias 3 -> 5
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
Commit message: Biblioteca Waveform
Parts:
- removed U$2: TSOP4838, tsop-1:TSOP18XX
- added Q5: TSOP4838, tsop:TSOP18XX
Connections:
- net GND: now also Q5.GND; no longer U$2.GND
- net VDD33: now also Q5.VCC; no longer U$2.VCC
- net VP_SENSOR_IR: now also Q5.OUT; no longer U$2.OUT
Routing:
- net GND: track 742.0 -> 746.4 mm, vias 47 -> 50
- net VP_SENSOR_IR: track 23.6 -> 22.8 mm
Changed lines of the file:
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@@
 <?xml version="1.0" encoding="utf-8"?>
 <!DOCTYPE eagle SYSTEM "eagle.dtd">
-<eagle version="9.6.2">
+<eagle version="9.5.1">
 <drawing>
 <settings>
@@
 <setting verticaltext="up"/>
 </settings>
-<grid distance="3.125" unitdist="mil" unit="mil" style="lines" multiple="1" display="yes" altdistance="5" altunitdist="mil" altunit="mil"/>
+<grid distance="6.25" unitdist="mil" unit="mil" style="lines" multiple="1" display="yes" altdistance="5" altunitdist="mil" altunit="mil"/>
 <layers>
 <layer number="1" name="Top" color="4" fill="1" visible="yes" active="yes"/>
@@
 <attribute name="VALUE" x="123.825" y="38.235" size="0.8128" layer="27" ratio="10" rot="R180"/>
 </element>
-<element name="U$2" library="tsop-1" package="TSOP18XX" value="TSOP4838" x="130.81" y="48.26" smashed="yes"/>
+<element name="Q5" library="tsop" package="TSOP18XX" value="TSOP4838" x="130.8512" y="47.333675" smashed="yes"/>
 </elements>
 <signals>
@@
 <contactref element="C17" pad="P-"/>
 <contactref element="C18" pad="P-"/>
-<contactref element="U$2" pad="GND"/>
+<contactref element="Q5" pad="GND"/>
 <wire x1="15.5575" y1="135.255" x2="13.49375" y2="135.255" width="0.2032" layer="1"/>
 <wire x1="18.57375" y1="138.27125" x2="15.5575" y2="135.255" width="0.2032" layer="1"/>
@@
 <wire x1="122.71375" y1="36.5125" x2="122.71375" y2="36.83" width="0.2032" layer="1"/>
 <wire x1="123.19" y1="36.03625" x2="122.71375" y2="36.5125" width="0.2032" layer="1"/>
-<wire x1="130.65125" y1="36.03625" x2="128.905" y2="36.03625" width="0.2032" layer="1"/>
-<wire x1="128.905" y1="36.03625" x2="123.19" y2="36.03625" width="0.2032" layer="1"/>
-<wire x1="131.1275" y1="36.5125" x2="130.65125" y2="36.03625" width="0.2032" layer="1"/>
+<wire x1="130.65125" y1="36.03625" x2="123.19" y2="36.03625" width="0.2032" layer="1"/>
+<wire x1="131.1275" y1="36.5125" x2="131.048125" y2="36.433125" width="0.2032" layer="1"/>
+<wire x1="131.048125" y1="36.433125" x2="130.65125" y2="36.03625" width="0.2032" layer="1"/>
 <wire x1="122.71375" y1="36.83" x2="122.69" y2="36.83" width="0.2032" layer="1"/>
 <wire x1="131.1275" y1="36.5125" x2="131.1275" y2="36.66875" width="0.2032" layer="1"/>
@@
 <wire x1="99.3775" y1="118.11" x2="103.8225" y2="113.665" width="0.2032" layer="16"/>
 <wire x1="92.7075" y1="118.11" x2="99.3775" y2="118.11" width="0.2032" layer="16"/>
-<wire x1="128.905" y1="46.355" x2="128.905" y2="36.03625" width="0.2032" layer="1"/>
-<wire x1="130.65125" y1="48.10125" x2="128.905" y2="46.355" width="0.2032" layer="1"/>
-<wire x1="130.65125" y1="48.10125" x2="130.8088" y2="48.2334" width="0.2032" layer="1"/>
 <wire x1="102.87" y1="121.6025" x2="102.87" y2="130.4925" width="0.2032" layer="1"/>
 <wire x1="99.3775" y1="118.11" x2="102.87" y2="121.6025" width="0.2032" layer="16"/>
@@
 <wire x1="123.95305625" y1="96.599375" x2="120.015" y2="96.599375" width="0.2032" layer="16"/>
 <wire x1="120.015" y1="96.599375" x2="119.38" y2="97.234375" width="0.2032" layer="16"/>
+<wire x1="130.85" y1="47.307075" x2="131.8663" y2="48.323375" width="0.2032" layer="1"/>
+<wire x1="131.8663" y1="48.323375" x2="131.9784" y2="48.323375" width="0.2032" layer="1"/>
+<via x="131.9784" y="48.323375" extent="1-16" drill="0.508"/>
+<wire x1="132.92915625" y1="48.983475" x2="132.962225" y2="48.983475" width="0.2032" layer="16"/>
+<wire x1="132.962225" y1="48.983475" x2="135.09625" y2="51.1175" width="0.2032" layer="16"/>
+<wire x1="131.9784" y1="48.323375" x2="132.26905625" y2="48.323375" width="0.2032" layer="16"/>
+<wire x1="132.26905625" y1="48.323375" x2="132.92915625" y2="48.983475" width="0.2032" layer="16"/>
+<wire x1="130.85" y1="47.307075" x2="130.199553125" y2="46.656628125" width="0.2032" layer="1"/>
+<wire x1="130.199553125" y1="46.656628125" x2="130.199553125" y2="45.377946875" width="0.2032" layer="1"/>
+<via x="130.199553125" y="45.377946875" extent="1-16" drill="0.6096"/>
+<wire x1="130.199553125" y1="45.377946875" x2="130.65125" y2="44.92625" width="0.2032" layer="16"/>
+<via x="130.65125" y="38.4175" extent="1-16" drill="0.6096"/>
+<wire x1="130.65125" y1="38.4175" x2="131.048125" y2="38.020625" width="0.2032" layer="1"/>
+<wire x1="131.048125" y1="38.020625" x2="131.048125" y2="36.433125" width="0.2032" layer="1"/>
+<wire x1="130.65125" y1="44.92625" x2="130.65125" y2="38.4175" width="0.2032" layer="16"/>
 </signal>
 <signal name="12(5V)">
@@
 <contactref element="V4" pad="9"/>
 <contactref element="V4" pad="12"/>
-<contactref element="U$2" pad="VCC"/>
+<contactref element="Q5" pad="VCC"/>
 <wire x1="130.81" y1="72.39" x2="127.79375" y2="75.40625" width="0.2032" layer="16"/>
 <wire x1="127.79375" y1="75.40625" x2="125.73" y2="77.47" width="0.2032" layer="16"/>
@@
 <wire x1="132.3975" y1="80.01" x2="127.79375" y2="75.40625" width="0.2032" layer="16"/>
 <wire x1="132.3975" y1="80.01" x2="133.35" y2="80.01" width="0.2032" layer="16"/>
-<wire x1="130.01625" y1="44.92625" x2="130.01625" y2="41.11625" width="0.2032" layer="1"/>
-<wire x1="133.19125" y1="48.10125" x2="130.01625" y2="44.92625" width="0.2032" layer="1"/>
+<wire x1="130.01625" y1="41.11625" x2="130.01625" y2="43.973325" width="0.2032" layer="1"/>
 <wire x1="130.01625" y1="41.11625" x2="129.86875" y2="41.11625" width="0.2032" layer="1"/>
-<wire x1="133.19125" y1="48.10125" x2="133.3088" y2="48.2334" width="0.2032" layer="1"/>
 <wire x1="118.745" y1="52.705" x2="116.84" y2="54.61" width="0.2032" layer="16"/>
 <wire x1="122.555" y1="52.705" x2="118.745" y2="52.705" width="0.2032" layer="16"/>
@@
 <wire x1="116.84" y1="54.61" x2="116.36375" y2="55.08625" width="0.2032" layer="16"/>
 <wire x1="69.69125" y1="56.1975" x2="69.611875" y2="56.1975" width="0.2032" layer="16"/>
-<wire x1="128.74625" y1="52.705" x2="133.19125" y2="48.26" width="0.2032" layer="1"/>
-<wire x1="126.365" y1="52.705" x2="128.74625" y2="52.705" width="0.2032" layer="1"/>
+<wire x1="128.5875" y1="52.705" x2="126.365" y2="52.705" width="0.2032" layer="1"/>
 <wire x1="124.46" y1="54.61" x2="126.365" y2="52.705" width="0.2032" layer="1"/>
-<wire x1="133.19125" y1="48.26" x2="133.3088" y2="48.2334" width="0.2032" layer="1"/>
 <wire x1="135.255" y1="70.485" x2="133.35" y2="72.39" width="0.2032" layer="16"/>
 <wire x1="135.255" y1="64.135" x2="135.255" y2="70.485" width="0.2032" layer="16"/>
@@
 <wire x1="133.19125" y1="107.15625" x2="134.540625" y2="108.505625" width="0.2032" layer="16"/>
 <wire x1="134.540625" y1="109.37875" x2="136.525" y2="107.394375" width="0.2032" layer="16"/>
+<wire x1="132.7912" y1="48.66005" x2="132.315075" y2="49.136175" width="0.2032" layer="1"/>
+<wire x1="133.35" y1="47.307075" x2="132.7912" y2="47.865875" width="0.2032" layer="1"/>
+<wire x1="132.7912" y1="47.865875" x2="132.7912" y2="48.66005" width="0.2032" layer="1"/>
+<wire x1="132.315075" y1="49.136175" x2="132.156325" y2="49.136175" width="0.2032" layer="1"/>
+<wire x1="132.156325" y1="49.136175" x2="128.5875" y2="52.705" width="0.2032" layer="1"/>
+<wire x1="130.01625" y1="43.973325" x2="133.35" y2="47.307075" width="0.2032" layer="1"/>
 </signal>
 <signal name="MOSI">
@@
 <wire x1="129.54" y1="52.54625" x2="129.54" y2="54.61" width="0.6096" layer="16"/>
 <wire x1="127.635" y1="52.54625" x2="129.54" y2="52.54625" width="0.6096" layer="16"/>
-<wire x1="125.57125" y1="50.4825" x2="127.635" y2="52.54625" width="0.6096" layer="16"/>
+<wire x1="125.57125" y1="50.4825" x2="127.555625" y2="52.466875" width="0.6096" layer="16"/>
+<wire x1="127.555625" y1="52.466875" x2="127.635" y2="52.54625" width="0.6096" layer="16"/>
 <wire x1="119.38" y1="50.4825" x2="125.57125" y2="50.4825" width="0.6096" layer="16"/>
 <wire x1="113.50625" y1="44.60875" x2="119.38" y2="50.4825" width="0.6096" layer="1"/>
@@
 <signal name="VP_SENSOR_IR">
 <contactref element="S4" pad="S"/>
-<contactref element="U$2" pad="OUT"/>
-<wire x1="128.42875" y1="28.41625" x2="128.42875" y2="48.10125" width="0.6096" layer="16"/>
+<contactref element="Q5" pad="OUT"/>
+<wire x1="128.42875" y1="28.41625" x2="128.42875" y2="47.344928125" width="0.6096" layer="16"/>
 <wire x1="129.69875" y1="28.41625" x2="128.42875" y2="28.41625" width="0.6096" layer="16"/>
 <wire x1="131.445" y1="26.67" x2="129.69875" y2="28.41625" width="0.6096" layer="16"/>
-<wire x1="128.42875" y1="48.10125" x2="128.3088" y2="48.2334" width="0.6096" layer="16"/>
+<wire x1="128.42875" y1="47.344928125" x2="128.35" y2="47.307075" width="0.6096" layer="16"/>
 </signal>
 <signal name="VIN1">
@@
 <wire x1="64.61125" y1="119.0625" x2="64.61125" y2="123.98375" width="0.6096" layer="1"/>
 <wire x1="62.865" y1="117.31625" x2="64.61125" y2="119.0625" width="0.6096" layer="1"/>
-<wire x1="62.865" y1="73.66" x2="62.865" y2="117.31625" width="0.6096" layer="1"/>
+<wire x1="62.865" y1="73.66" x2="62.865" y2="95.25" width="0.6096" layer="1"/>
+<wire x1="62.865" y1="95.25" x2="62.865" y2="117.31625" width="0.6096" layer="1"/>
 <wire x1="60.96" y1="71.755" x2="62.865" y2="73.66" width="0.6096" layer="1"/>
 <wire x1="60.96" y1="67.945" x2="60.96" y2="71.755" width="0.6096" layer="1"/>
